File: hw/remote-io-can.sch (KiCad schematic (older format))
At the start: 13 parts, among them U6 MCP2515, U7 ADM3054, Y1 Crystal

Commit message: Started fucking aroond with pcb layout. Power is tricky...
Changed lines of the file:
@@
 $EndComp
 $Comp
-L GND #PWR062
+L GND #PWR059
 U 1 1 5581E9B9
 P 8400 4900
-F 0 "#PWR062" H 8400 4650 50  0001 C CNN
+F 0 "#PWR059" H 8400 4650 50  0001 C CNN
 F 1 "GND" H 8400 4750 50  0000 C CNN
 F 2 "" H 8400 4900 60  0000 C CNN
@@
 $EndComp
 $Comp
-L GND #PWR063
+L GND #PWR060
 U 1 1 5581E9D3
 P 7050 4900
-F 0 "#PWR063" H 7050 4650 50  0001 C CNN
+F 0 "#PWR060" H 7050 4650 50  0001 C CNN
 F 1 "GND" H 7050 4750 50  0000 C CNN
 F 2 "" H 7050 4900 60  0000 C CNN
@@
 Connection ~ 8400 4850
 $Comp
-L +5VA #PWR064
+L +5VA #PWR061
 U 1 1 5581F152
 P 8400 4000
-F 0 "#PWR064" H 8400 3850 50  0001 C CNN
+F 0 "#PWR061" H 8400 3850 50  0001 C CNN
 F 1 "+5VA" H 8400 4140 50  0000 C CNN
 F 2 "" H 8400 4000 60  0000 C CNN
@@
 $EndComp
 $Comp
-L GND #PWR065
+L GND #PWR062
 U 1 1 5581F4D8
 P 8050 3350
-F 0 "#PWR065" H 8050 3100 50  0001 C CNN
+F 0 "#PWR062" H 8050 3100 50  0001 C CNN
 F 1 "GND" H 8050 3200 50  0000 C CNN
 F 2 "" H 8050 3350 60  0000 C CNN
@@
 $EndComp
 $Comp
-L +5VA #PWR066
+L +5VA #PWR063
 U 1 1 5581F526
 P 8050 3050
-F 0 "#PWR066" H 8050 2900 50  0001 C CNN
+F 0 "#PWR063" H 8050 2900 50  0001 C CNN
 F 1 "+5VA" H 8050 3190 50  0000 C CNN
 F 2 "" H 8050 3050 60  0000 C CNN
@@
 $EndComp
 $Comp
-L +3.3V #PWR067
+L +3.3V #PWR064
 U 1 1 5581F57B
 P 7400 3050
-F 0 "#PWR067" H 7400 2900 50  0001 C CNN
+F 0 "#PWR064" H 7400 2900 50  0001 C CNN
 F 1 "+3.3V" H 7400 3190 50  0000 C CNN
 F 2 "" H 7400 3050 60  0000 C CNN
@@
 $EndComp
 $Comp
-L GND #PWR068
+L GND #PWR065
 U 1 1 5581F5A8
 P 7400 3350
-F 0 "#PWR068" H 7400 3100 50  0001 C CNN
+F 0 "#PWR065" H 7400 3100 50  0001 C CNN
 F 1 "GND" H 7400 3200 50  0000 C CNN
 F 2 "" H 7400 3350 60  0000 C CNN
@@
 $EndComp
 $Comp
-L +3.3V #PWR069
+L +3.3V #PWR066
 U 1 1 5581F6ED
 P 7050 4000
-F 0 "#PWR069" H 7050 3850 50  0001 C CNN
+F 0 "#PWR066" H 7050 3850 50  0001 C CNN
 F 1 "+3.3V" H 7050 4140 50  0000 C CNN
 F 2 "" H 7050 4000 60  0000 C CNN
@@
 $EndComp
 $Comp
-L GND #PWR070
+L GND #PWR067
 U 1 1 5582103F
 P 9050 4550
-F 0 "#PWR070" H 9050 4300 50  0001 C CNN
+F 0 "#PWR067" H 9050 4300 50  0001 C CNN
 F 1 "GND" H 9050 4400 50  0000 C CNN
 F 2 "" H 9050 4550 60  0000 C CNN
@@
 Connection ~ 5000 3450
 $Comp
-L GND #PWR071
+L GND #PWR068
 U 1 1 55822EB0
 P 5150 3500
-F 0 "#PWR071" H 5150 3250 50  0001 C CNN
+F 0 "#PWR068" H 5150 3250 50  0001 C CNN
 F 1 "GND" H 5150 3350 50  0000 C CNN
 F 2 "" H 5150 3500 60  0000 C CNN
@@
 NoConn ~ 2200 4350
 $Comp
-L GND #PWR072
+L GND #PWR069
 U 1 1 55825BA2
 P 2200 4550
-F 0 "#PWR072" H 2200 4300 50  0001 C CNN
+F 0 "#PWR069" H 2200 4300 50  0001 C CNN
 F 1 "GND" H 2200 4400 50  0000 C CNN
 F 2 "" H 2200 4550 60  0000 C CNN
@@
 	3800 4500 3900 4500
 $Comp
-L +3.3V #PWR073
+L +3.3V #PWR070
 U 1 1 5584B17B
 P 1950 3150
-F 0 "#PWR073" H 1950 3000 50  0001 C CNN
+F 0 "#PWR070" H 1950 3000 50  0001 C CNN
 F 1 "+3.3V" H 1950 3290 50  0000 C CNN
 F 2 "" H 1950 3150 60  0000 C CNN
@@
 $EndComp
 $Comp
-L +3.3V #PWR074
+L +3.3V #PWR071
 U 1 1 5584D12C
 P 1550 4150
-F 0 "#PWR074" H 1550 4000 50  0001 C CNN
+F 0 "#PWR071" H 1550 4000 50  0001 C CNN
 F 1 "+3.3V" H 1550 4290 50  0000 C CNN
 F 2 "" H 1550 4150 60  0000 C CNN
@@
 $EndComp
 $Comp
-L GND #PWR075
+L GND #PWR072
 U 1 1 5584D132
 P 1550 4450
-F 0 "#PWR075" H 1550 4200 50  0001 C CNN
+F 0 "#PWR072" H 1550 4200 50  0001 C CNN
 F 1 "GND" H 1550 4300 50  0000 C CNN
 F 2 "" H 1550 4450 60  0000 C CNN
@@
 Text HLabel 7050 4100 0    60   Output ~ 0
 CAN_VSENSE
+Connection ~ 2200 4550
+Connection ~ 1550 4450
+Connection ~ 5150 3500
+Connection ~ 7050 4900
+Connection ~ 8400 4900
+Connection ~ 9050 4550
+Connection ~ 8050 3350
+Connection ~ 7400 3350
 $EndSCHEMATC

Commit message: All parts in hat-spec-size board
Changed lines of the file:
@@
 $Descr A4 11693 8268
 encoding utf-8
-Sheet 6 6
+Sheet 5 5
 Title ""
 Date ""
@@
 $EndComp
 $Comp
-L GND #PWR059
+L GND #PWR053
 U 1 1 5581E9B9
 P 8400 4900
-F 0 "#PWR059" H 8400 4650 50  0001 C CNN
+F 0 "#PWR053" H 8400 4650 50  0001 C CNN
 F 1 "GND" H 8400 4750 50  0000 C CNN
 F 2 "" H 8400 4900 60  0000 C CNN
@@
 $EndComp
 $Comp
-L GND #PWR060
+L GND #PWR054
 U 1 1 5581E9D3
 P 7050 4900
-F 0 "#PWR060" H 7050 4650 50  0001 C CNN
+F 0 "#PWR054" H 7050 4650 50  0001 C CNN
 F 1 "GND" H 7050 4750 50  0000 C CNN
 F 2 "" H 7050 4900 60  0000 C CNN
@@
 Connection ~ 8400 4850
 $Comp
-L +5VA #PWR061
+L +5VA #PWR055
 U 1 1 5581F152
 P 8400 4000
-F 0 "#PWR061" H 8400 3850 50  0001 C CNN
+F 0 "#PWR055" H 8400 3850 50  0001 C CNN
 F 1 "+5VA" H 8400 4140 50  0000 C CNN
 F 2 "" H 8400 4000 60  0000 C CNN
@@
 $EndComp
 $Comp
-L GND #PWR062
+L GND #PWR056
 U 1 1 5581F4D8
 P 8050 3350
-F 0 "#PWR062" H 8050 3100 50  0001 C CNN
+F 0 "#PWR056" H 8050 3100 50  0001 C CNN
 F 1 "GND" H 8050 3200 50  0000 C CNN
 F 2 "" H 8050 3350 60  0000 C CNN
@@
 $EndComp
 $Comp
-L +5VA #PWR063
+L +5VA #PWR057
 U 1 1 5581F526
 P 8050 3050
-F 0 "#PWR063" H 8050 2900 50  0001 C CNN
+F 0 "#PWR057" H 8050 2900 50  0001 C CNN
 F 1 "+5VA" H 8050 3190 50  0000 C CNN
 F 2 "" H 8050 3050 60  0000 C CNN
@@
 $EndComp
 $Comp
-L +3.3V #PWR064
+L +3.3V #PWR058
 U 1 1 5581F57B
 P 7400 3050
-F 0 "#PWR064" H 7400 2900 50  0001 C CNN
+F 0 "#PWR058" H 7400 2900 50  0001 C CNN
 F 1 "+3.3V" H 7400 3190 50  0000 C CNN
 F 2 "" H 7400 3050 60  0000 C CNN
@@
 $EndComp
 $Comp
-L GND #PWR065
+L GND #PWR059
 U 1 1 5581F5A8
 P 7400 3350
-F 0 "#PWR065" H 7400 3100 50  0001 C CNN
+F 0 "#PWR059" H 7400 3100 50  0001 C CNN
 F 1 "GND" H 7400 3200 50  0000 C CNN
 F 2 "" H 7400 3350 60  0000 C CNN
@@
 $EndComp
 $Comp
-L +3.3V #PWR066
+L +3.3V #PWR060
 U 1 1 5581F6ED
 P 7050 4000
-F 0 "#PWR066" H 7050 3850 50  0001 C CNN
+F 0 "#PWR060" H 7050 3850 50  0001 C CNN
 F 1 "+3.3V" H 7050 4140 50  0000 C CNN
 F 2 "" H 7050 4000 60  0000 C CNN
@@
 $EndComp
 $Comp
-L GND #PWR067
+L GND #PWR061
 U 1 1 5582103F
 P 9050 4550
-F 0 "#PWR067" H 9050 4300 50  0001 C CNN
+F 0 "#PWR061" H 9050 4300 50  0001 C CNN
 F 1 "GND" H 9050 4400 50  0000 C CNN
 F 2 "" H 9050 4550 60  0000 C CNN
@@
 Connection ~ 5000 3450
 $Comp
-L GND #PWR068
+L GND #PWR062
 U 1 1 55822EB0
 P 5150 3500
-F 0 "#PWR068" H 5150 3250 50  0001 C CNN
+F 0 "#PWR062" H 5150 3250 50  0001 C CNN
 F 1 "GND" H 5150 3350 50  0000 C CNN
 F 2 "" H 5150 3500 60  0000 C CNN
@@
 NoConn ~ 2200 4350
 $Comp
-L GND #PWR069
+L GND #PWR063
 U 1 1 55825BA2
 P 2200 4550
-F 0 "#PWR069" H 2200 4300 50  0001 C CNN
+F 0 "#PWR063" H 2200 4300 50  0001 C CNN
 F 1 "GND" H 2200 4400 50  0000 C CNN
 F 2 "" H 2200 4550 60  0000 C CNN
@@
 	3800 4500 3900 4500
 $Comp
-L +3.3V #PWR070
+L +3.3V #PWR064
 U 1 1 5584B17B
 P 1950 3150
-F 0 "#PWR070" H 1950 3000 50  0001 C CNN
+F 0 "#PWR064" H 1950 3000 50  0001 C CNN
 F 1 "+3.3V" H 1950 3290 50  0000 C CNN
 F 2 "" H 1950 3150 60  0000 C CNN
@@
 $EndComp
 $Comp
-L +3.3V #PWR071
+L +3.3V #PWR065
 U 1 1 5584D12C
 P 1550 4150
-F 0 "#PWR071" H 1550 4000 50  0001 C CNN
+F 0 "#PWR065" H 1550 4000 50  0001 C CNN
 F 1 "+3.3V" H 1550 4290 50  0000 C CNN
 F 2 "" H 1550 4150 60  0000 C CNN
@@
 $EndComp
 $Comp
-L GND #PWR072
+L GND #PWR066
 U 1 1 5584D132
 P 1550 4450
-F 0 "#PWR072" H 1550 4200 50  0001 C CNN
+F 0 "#PWR066" H 1550 4200 50  0001 C CNN
 F 1 "GND" H 1550 4300 50  0000 C CNN
 F 2 "" H 1550 4450 60  0000 C CNN
@@
 Connection ~ 8050 3350
 Connection ~ 7400 3350
+Connection ~ 7400 3050
+Connection ~ 8050 3050
 $EndSCHEMATC

Commit message: Isolated CAN bus connections and added proper mounting holes
Connections:
- net GND: no longer C13.2, C9.2, U7.16 (GND2), U7.9 (GND2)
- new net GNDA: C13.2, C9.2, U7.16 (GND2), U7.9 (GND2)
Changed lines of the file:
@@
 EESchema Schematic File Version 2
+LIBS:remote-io-rescue
 LIBS:power
 LIBS:device
@@
 $EndComp
 $Comp
-L GND #PWR055
-U 1 1 5581E9B9
-P 8400 4900
-F 0 "#PWR055" H 8400 4650 50  0001 C CNN
-F 1 "GND" H 8400 4750 50  0000 C CNN
-F 2 "" H 8400 4900 60  0000 C CNN
-F 3 "" H 8400 4900 60  0000 C CNN
-	1    8400 4900
-	1    0    0    -1
-$EndComp
-$Comp
-L GND #PWR056
+L GND #PWR059
 U 1 1 5581E9D3
 P 7050 4900
-F 0 "#PWR056" H 7050 4650 50  0001 C CNN
+F 0 "#PWR059" H 7050 4650 50  0001 C CNN
 F 1 "GND" H 7050 4750 50  0000 C CNN
 F 2 "" H 7050 4900 60  0000 C CNN
@@
 Connection ~ 8400 4850
 $Comp
-L +5VA #PWR057
+L +5VA #PWR060
 U 1 1 5581F152
 P 8400 4000
-F 0 "#PWR057" H 8400 3850 50  0001 C CNN
+F 0 "#PWR060" H 8400 3850 50  0001 C CNN
 F 1 "+5VA" H 8400 4140 50  0000 C CNN
 F 2 "" H 8400 4000 60  0000 C CNN
@@
 $EndComp
 $Comp
-L GND #PWR058
-U 1 1 5581F4D8
-P 8050 3350
-F 0 "#PWR058" H 8050 3100 50  0001 C CNN
-F 1 "GND" H 8050 3200 50  0000 C CNN
-F 2 "" H 8050 3350 60  0000 C CNN
-F 3 "" H 8050 3350 60  0000 C CNN
-	1    8050 3350
-	1    0    0    -1
-$EndComp
-$Comp
-L +5VA #PWR059
+L +5VA #PWR061
 U 1 1 5581F526
 P 8050 3050
-F 0 "#PWR059" H 8050 2900 50  0001 C CNN
+F 0 "#PWR061" H 8050 2900 50  0001 C CNN
 F 1 "+5VA" H 8050 3190 50  0000 C CNN
 F 2 "" H 8050 3050 60  0000 C CNN
@@
 $EndComp
 $Comp
-L +3.3V #PWR060
+L +3.3V #PWR062
 U 1 1 5581F57B
 P 7400 3050
-F 0 "#PWR060" H 7400 2900 50  0001 C CNN
+F 0 "#PWR062" H 7400 2900 50  0001 C CNN
 F 1 "+3.3V" H 7400 3190 50  0000 C CNN
 F 2 "" H 7400 3050 60  0000 C CNN
@@
 $EndComp
 $Comp
-L GND #PWR061
+L GND #PWR063
 U 1 1 5581F5A8
 P 7400 3350
-F 0 "#PWR061" H 7400 3100 50  0001 C CNN
+F 0 "#PWR063" H 7400 3100 50  0001 C CNN
 F 1 "GND" H 7400 3200 50  0000 C CNN
 F 2 "" H 7400 3350 60  0000 C CNN
@@
 $EndComp
 $Comp
-L +3.3V #PWR062
+L +3.3V #PWR064
 U 1 1 5581F6ED
 P 7050 4000
-F 0 "#PWR062" H 7050 3850 50  0001 C CNN
+F 0 "#PWR064" H 7050 3850 50  0001 C CNN
 F 1 "+3.3V" H 7050 4140 50  0000 C CNN
 F 2 "" H 7050 4000 60  0000 C CNN
@@
 	1    9200 4350
 	0    1    1    0
-$EndComp
-$Comp
-L GND #PWR063
-U 1 1 5582103F
-P 9050 4550
-F 0 "#PWR063" H 9050 4300 50  0001 C CNN
-F 1 "GND" H 9050 4400 50  0000 C CNN
-F 2 "" H 9050 4550 60  0000 C CNN
-F 3 "" H 9050 4550 60  0000 C CNN
-	1    9050 4550
-	1    0    0    -1
 $EndComp
 Wire Wire Line
@@
 Connection ~ 5000 3450
 $Comp
-L GND #PWR064
+L GND #PWR065
 U 1 1 55822EB0
 P 5150 3500
-F 0 "#PWR064" H 5150 3250 50  0001 C CNN
+F 0 "#PWR065" H 5150 3250 50  0001 C CNN
 F 1 "GND" H 5150 3350 50  0000 C CNN
 F 2 "" H 5150 3500 60  0000 C CNN
@@
 NoConn ~ 2200 4350
 $Comp
-L GND #PWR065
+L GND #PWR066
 U 1 1 55825BA2
 P 2200 4550
-F 0 "#PWR065" H 2200 4300 50  0001 C CNN
+F 0 "#PWR066" H 2200 4300 50  0001 C CNN
 F 1 "GND" H 2200 4400 50  0000 C CNN
 F 2 "" H 2200 4550 60  0000 C CNN
@@
 	3800 4500 3900 4500
 $Comp
-L +3.3V #PWR066
+L +3.3V #PWR067
 U 1 1 5584B17B
 P 1950 3150
-F 0 "#PWR066" H 1950 3000 50  0001 C CNN
+F 0 "#PWR067" H 1950 3000 50  0001 C CNN
 F 1 "+3.3V" H 1950 3290 50  0000 C CNN
 F 2 "" H 1950 3150 60  0000 C CNN
@@
 $EndComp
 $Comp
-L +3.3V #PWR067
+L +3.3V #PWR068
 U 1 1 5584D12C
 P 1550 4150
-F 0 "#PWR067" H 1550 4000 50  0001 C CNN
+F 0 "#PWR068" H 1550 4000 50  0001 C CNN
 F 1 "+3.3V" H 1550 4290 50  0000 C CNN
 F 2 "" H 1550 4150 60  0000 C CNN
@@
 $EndComp
 $Comp
-L GND #PWR068
+L GND #PWR069
 U 1 1 5584D132
 P 1550 4450
-F 0 "#PWR068" H 1550 4200 50  0001 C CNN
+F 0 "#PWR069" H 1550 4200 50  0001 C CNN
 F 1 "GND" H 1550 4300 50  0000 C CNN
 F 2 "" H 1550 4450 60  0000 C CNN
@@
 Connection ~ 5150 3500
 Connection ~ 7050 4900
-Connection ~ 8400 4900
-Connection ~ 9050 4550
-Connection ~ 8050 3350
 Connection ~ 7400 3350
 Connection ~ 7400 3050
 Connection ~ 8050 3050
+$Comp
+L GNDA #PWR070
+U 1 1 558B0993
+P 8400 4900
+F 0 "#PWR070" H 8400 4650 50  0001 C CNN
+F 1 "GNDA" H 8400 4750 50  0000 C CNN
+F 2 "" H 8400 4900 60  0000 C CNN
+F 3 "" H 8400 4900 60  0000 C CNN
+	1    8400 4900
+	1    0    0    -1
+$EndComp
+$Comp
+L GNDA #PWR071
+U 1 1 558B0A40
+P 9050 4550
+F 0 "#PWR071" H 9050 4300 50  0001 C CNN
+F 1 "GNDA" H 9050 4400 50  0000 C CNN
+F 2 "" H 9050 4550 60  0000 C CNN
+F 3 "" H 9050 4550 60  0000 C CNN
+	1    9050 4550
+	1    0    0    -1
+$EndComp
+Connection ~ 9050 4550
+Connection ~ 8400 4900
+$Comp
+L GNDA #PWR072
+U 1 1 558B0FA4
+P 8050 3350
+F 0 "#PWR072" H 8050 3100 50  0001 C CNN
+F 1 "GNDA" H 8050 3200 50  0000 C CNN
+F 2 "" H 8050 3350 60  0000 C CNN
+F 3 "" H 8050 3350 60  0000 C CNN
+	1    8050 3350
+	1    0    0    -1
+$EndComp
+Connection ~ 8050 3350
 $EndSCHEMATC
