File: hw/remote-io-power.sch (KiCad schematic (older format))
At the start: 16 parts, among them Q1 DMG2305UX, Q2 DMMT5401, U1 AP1506, U2 LP2992

Commit message: Isolated CAN bus connections and added proper mounting holes
Parts:
- U1: symbol AP1506 -> AP1506-RESCUE-remote-io
Connections:
- net +12V: no longer D6.1 (K), U2.1 (VIN), U2.3 (ON/~OFF)
- net GND: no longer C3.2, C4.2, U2.2 (GND)
- new net +12VA: D6.1 (K), U2.1 (VIN), U2.3 (ON/~OFF)
- new net GNDA: C3.2, C4.2, U2.2 (GND)
Changed lines of the file:
@@
 EESchema Schematic File Version 2
+LIBS:remote-io-rescue
 LIBS:power
 LIBS:device
@@
 $EndDescr
 $Comp
-L AP1506 U1
+L AP1506-RESCUE-remote-io U1
 U 1 1 557EE55F
 P 3800 3550
+AR Path="/557EE55F" Ref="U1"  Part="1"
+AR Path="/557F39A6/557EE55F" Ref="U1"  Part="1"
 F 0 "U1" H 3700 3850 60  0000 C CNN
 F 1 "AP1506" H 3800 3750 60  0000 C CNN
@@
 Ideal Diode Circuit
 $Comp
-L +12V #PWR029
+L +12V #PWR033
 U 1 1 557F7629
 P 2950 3450
-F 0 "#PWR029" H 2950 3300 50  0001 C CNN
+F 0 "#PWR033" H 2950 3300 50  0001 C CNN
 F 1 "+12V" H 2950 3590 50  0000 C CNN
 F 2 "" H 2950 3450 60  0000 C CNN
@@
 $EndComp
 $Comp
-L +5V #PWR030
+L +5V #PWR034
 U 1 1 557F764F
 P 7750 3000
-F 0 "#PWR030" H 7750 2850 50  0001 C CNN
+F 0 "#PWR034" H 7750 2850 50  0001 C CNN
 F 1 "+5V" H 7750 3140 50  0000 C CNN
 F 2 "" H 7750 3000 60  0000 C CNN
@@
 V_GATE
 $Comp
-L GND #PWR031
+L GND #PWR035
 U 1 1 5582FAEC
 P 5050 3900
-F 0 "#PWR031" H 5050 3650 50  0001 C CNN
+F 0 "#PWR035" H 5050 3650 50  0001 C CNN
 F 1 "GND" H 5050 3750 50  0000 C CNN
 F 2 "" H 5050 3900 60  0000 C CNN
@@
 $EndComp
 $Comp
-L GND #PWR032
+L GND #PWR036
 U 1 1 5582FB3E
 P 6550 4700
-F 0 "#PWR032" H 6550 4450 50  0001 C CNN
+F 0 "#PWR036" H 6550 4450 50  0001 C CNN
 F 1 "GND" H 6550 4550 50  0000 C CNN
 F 2 "" H 6550 4700 60  0000 C CNN
@@
 $EndComp
 $Comp
-L GND #PWR033
+L GND #PWR037
 U 1 1 5582FB61
 P 7200 4650
-F 0 "#PWR033" H 7200 4400 50  0001 C CNN
+F 0 "#PWR037" H 7200 4400 50  0001 C CNN
 F 1 "GND" H 7200 4500 50  0000 C CNN
 F 2 "" H 7200 4650 60  0000 C CNN
@@
 $EndComp
 $Comp
-L GND #PWR034
+L GND #PWR038
 U 1 1 5582FB89
 P 5800 3000
-F 0 "#PWR034" H 5800 2750 50  0001 C CNN
+F 0 "#PWR038" H 5800 2750 50  0001 C CNN
 F 1 "GND" H 5800 2850 50  0000 C CNN
 F 2 "" H 5800 3000 60  0000 C CNN
@@
 $EndComp
 $Comp
-L GND #PWR035
+L GND #PWR039
 U 1 1 5582FBB1
 P 7900 4150
-F 0 "#PWR035" H 7900 3900 50  0001 C CNN
+F 0 "#PWR039" H 7900 3900 50  0001 C CNN
 F 1 "GND" H 7900 4000 50  0000 C CNN
 F 2 "" H 7900 4150 60  0000 C CNN
@@
 	1    0    0    -1
 $EndComp
-$Comp
-L GND #PWR036
-U 1 1 5584C204
-P 3850 6600
-F 0 "#PWR036" H 3850 6350 50  0001 C CNN
-F 1 "GND" H 3850 6450 50  0000 C CNN
-F 2 "" H 3850 6600 60  0000 C CNN
-F 3 "" H 3850 6600 60  0000 C CNN
-	1    3850 6600
-	1    0    0    -1
-$EndComp
 Wire Wire Line
 	3600 6300 3650 6300
@@
 Connection ~ 2300 6100
 $Comp
-L GND #PWR037
-U 1 1 5584C221
-P 2300 6300
-F 0 "#PWR037" H 2300 6050 50  0001 C CNN
-F 1 "GND" H 2300 6150 50  0000 C CNN
-F 2 "" H 2300 6300 60  0000 C CNN
-F 3 "" H 2300 6300 60  0000 C CNN
-	1    2300 6300
-	1    0    0    -1
-$EndComp
-$Comp
-L +5VA #PWR038
+L +5VA #PWR040
 U 1 1 5584C227
 P 3900 6100
-F 0 "#PWR038" H 3900 5950 50  0001 C CNN
+F 0 "#PWR040" H 3900 5950 50  0001 C CNN
 F 1 "+5VA" H 3900 6240 50  0000 C CNN
 F 2 "" H 3900 6100 60  0000 C CNN
@@
 Text Notes 2050 5400 0    60   ~ 0
 CAN Transciever Power Supply
-$Comp
-L +12V #PWR039
-U 1 1 55852018
-P 2150 6100
-F 0 "#PWR039" H 2150 5950 50  0001 C CNN
-F 1 "+12V" H 2150 6240 50  0000 C CNN
-F 2 "" H 2150 6100 60  0000 C CNN
-F 3 "" H 2150 6100 60  0000 C CNN
-	1    2150 6100
-	1    0    0    -1
-$EndComp
 Wire Wire Line
 	2150 6100 2300 6100
 Connection ~ 5050 3900
-Connection ~ 3850 6600
 Connection ~ 3900 6100
-Connection ~ 2300 6300
 Connection ~ 7200 4650
 Connection ~ 7750 3000
@@
 Connection ~ 6550 4700
 Connection ~ 3400 3650
+$Comp
+L GNDA #PWR041
+U 1 1 558B302B
+P 2300 6300
+F 0 "#PWR041" H 2300 6050 50  0001 C CNN
+F 1 "GNDA" H 2300 6150 50  0000 C CNN
+F 2 "" H 2300 6300 60  0000 C CNN
+F 3 "" H 2300 6300 60  0000 C CNN
+	1    2300 6300
+	1    0    0    -1
+$EndComp
+$Comp
+L +12VA #PWR042
+U 1 1 558B305F
+P 2150 6100
+F 0 "#PWR042" H 2150 5950 50  0001 C CNN
+F 1 "+12VA" H 2150 6240 50  0000 C CNN
+F 2 "" H 2150 6100 60  0000 C CNN
+F 3 "" H 2150 6100 60  0000 C CNN
+	1    2150 6100
+	1    0    0    -1
+$EndComp
+$Comp
+L GNDA #PWR043
+U 1 1 558B3451
+P 3850 6600
+F 0 "#PWR043" H 3850 6350 50  0001 C CNN
+F 1 "GNDA" H 3850 6450 50  0000 C CNN
+F 2 "" H 3850 6600 60  0000 C CNN
+F 3 "" H 3850 6600 60  0000 C CNN
+	1    3850 6600
+	1    0    0    -1
+$EndComp
+Connection ~ 3850 6600
+Connection ~ 2300 6300
+Connection ~ 2150 6100
 $EndSCHEMATC
